File: ecg.kicad_sch (KiCad schematic)
At the start: 24 parts, among them SW1 SW_Push, SW2 SW_Push, U1 ESP32-S3-PICO-1-N8R2, U2 AD620, U3 OPA358

Commit message: Tinker with Antenna ckt
Parts:
- removed AN1: ~, symbol antenna_ecg:Antenna_Blackbox
- added AE1, AE2: Antenna_Shield, Connector_Coaxial:U.FL_Hirose_U.FL-R-SMT-1_Vertical, symbol Device:Antenna_Shield
- added C7: 0.8 pF, Capacitor_SMD:C_0402_1005Metric, symbol Device:C
- added L1: 3.9 nH, Inductor_SMD:L_0402_1005Metric, symbol Device:L
- added R6: 100, Resistor_SMD:R_0201_0603Metric, symbol Device:R
- C4: value 0.1uF -> 1uF
- R2: value 0 -> 10k
- SW1, SW2: footprint (none) -> Button_Switch_THT:SW_PUSH_6mm_H5mm
Connections:
- net GND: now also AE2.2 (Shield), C7.2
- net RXD0: now also AE1.2 (Shield)
- net TMS: now also AE1.1 (A)
- net at C4.2, R2.1: now also R6.1; no longer SW1.2
- new net: AE2.1 (A), L1.1
- new net: C7.1, L1.2
- new net: R6.2, SW1.2
Other:
- note removed: "A push switch here"
- moved on the sheet: C11, C12, L2, R2, SW1
